Commit message: corrected xacro

File: ros2_dual_stepper_controller/description/urdf/dual_stepper.ros2_control.xacro (robot description, xacro)
@@ -1,3 +1,4 @@
 <?xml version="1.0"?>
+<robot xmlns:xacro="http://ros.org/wiki/xacro">
 <xacro:macro xmlns:xacro="http://www.ros.org/wiki/xacro" name="ros2_dual_stepper_controller" params="name">
     <ros2_control name="${name}" type="system">
@@ -7,10 +8,10 @@
             <param name="baud_rate">115200</param>
         </hardware>
-        <joint name="$left_wheel_joint">
+        <joint name="left_wheel_joint">
             <command_interface name="velocity"/>
             <state_interface name="position"/>
             <state_interface name="velocity"/>
         </joint>
-        <joint name="$right_wheel_joint">
+        <joint name="right_wheel_joint">
             <command_interface name="velocity"/>
             <state_interface name="position"/>
@@ -19,2 +20,3 @@
     </ros2_control>
 </xacro:macro>
+</robot>

File: ros2_dual_stepper_controller/description/urdf/dual_stepper.urdf.xacro (robot description, xacro)
@@ -1,8 +1,8 @@
 <?xml version="1.0"?>
-<robot xmlns:xacro="http://ros.org/wiki/xacro" name="dual_stepper">
+<robot xmlns:xacro="http://www.ros.org/wiki/xacro" name="dual_stepper">
     <!-- Include all macro definitions -->
-    <xacro:include filename="$(find ros2_dual_stepper_controller)/description/urdf/robot_parts/base_link.xacro"/>
-    <xacro:include filename="$(find ros2_dual_stepper_controller)/description/urdf/robot_parts/wheel.xacro"/>
-    <xacro:include filename="$(find ros2_dual_stepper_controller)/description/urdf/dual_stepper.ros2_control.xacro"/>
+    <xacro:include filename="robot_parts/base_link.xacro"/>
+    <xacro:include filename="robot_parts/wheel.xacro"/>
+    <xacro:include filename="dual_stepper.ros2_control.xacro"/>
     <!-- Define reusable materials -->
     <material name="grey">
@@ -14,8 +14,8 @@
     <!-- Robot structure -->
     <xacro:base_link/>
-    <xacro:wheel name="left_wheel" parent="base_link"
+    <xacro:wheel wheel_name="left_wheel" parent="base_link"
             xyz="-0.1156 0.0 0.046" rpy="0 0 0" axis="0 1 0"/>
-    <xacro:wheel name="right_wheel" parent="base_link"
-            xyz="0.1156 -0.0 0.04698" rpy="0 ${pi} 0" axis="0 1 0"/>
+    <xacro:wheel wheel_name="right_wheel" parent="base_link"
+            xyz="0.1156 0.0 0.046" rpy="0 ${pi} 0" axis="0 1 0"/>
     <xacro:ros2_dual_stepper_controller name="DualStepperSystem" />
 </robot>

File: ros2_dual_stepper_controller/description/urdf/robot_parts/base_link.xacro (robot description, xacro)
@@ -1,3 +1,4 @@
 <?xml version="1.0"?>
+<robot xmlns:xacro="http://ros.org/wiki/xacro">
 <xacro:macro name="base_link" xmlns:xacro="http://ros.org/wiki/xacro">
     <link name="base_link">
@@ -18,2 +19,3 @@
     </link>
 </xacro:macro>
+</robot>

File: ros2_dual_stepper_controller/description/urdf/robot_parts/wheel.xacro (robot description, xacro)
@@ -1,5 +1,6 @@
 <?xml version="1.0"?>
-<xacro:macro name="wheel" params="name parent xyz rpy axis" xmlns:xacro="http://ros.org/wiki/xacro">
-    <link name="${name}">
+<robot xmlns:xacro="http://ros.org/wiki/xacro">
+<xacro:macro name="wheel" params="wheel_name parent xyz rpy axis" xmlns:xacro="http://ros.org/wiki/xacro">
+    <link name="${wheel_name}">
         <visual>
             <origin rpy="0.0 0.0 0.0" xyz="0.0 0.0 0.0"/>
@@ -17,9 +18,10 @@
         </inertial>
     </link>
-    <joint name="${name}_joint" type="continuous">
+    <joint name="${wheel_name}_joint" type="continuous">
         <parent link="${parent}"/>
-        <child link="${name}"/>
+        <child link="${wheel_name}"/>
         <origin xyz="${xyz}" rpy="${rpy}"/>
         <axis xyz="${axis}"/>
     </joint>
 </xacro:macro>
+</robot>

Commit message: added launch and config

File: ros2_dual_stepper_controller/description/urdf/dual_stepper.ros2_control.xacro (robot description, xacro)
@@ -1,22 +1,22 @@
 <?xml version="1.0"?>
 <robot xmlns:xacro="http://ros.org/wiki/xacro">
-<xacro:macro xmlns:xacro="http://www.ros.org/wiki/xacro" name="ros2_dual_stepper_controller" params="name">
-    <ros2_control name="${name}" type="system">
-        <hardware>
-            <plugin>ros2_dual_stepper_controller/DualStepperHardwareInterface</plugin>
-            <param name="serial_port">/dev/ttyUSB0</param>
-            <param name="baud_rate">115200</param>
-        </hardware>
-        <joint name="left_wheel_joint">
-            <command_interface name="velocity"/>
-            <state_interface name="position"/>
-            <state_interface name="velocity"/>
-        </joint>
-        <joint name="right_wheel_joint">
-            <command_interface name="velocity"/>
-            <state_interface name="position"/>
-            <state_interface name="velocity"/>
-        </joint>
-    </ros2_control>
-</xacro:macro>
+    <xacro:macro name="ros2_dual_stepper_controller" params="name left right">
+        <ros2_control name="${name}" type="system">
+            <hardware>
+                <plugin>ros2_dual_stepper_controller/DualStepperHardwareInterface</plugin>
+                <param name="serial_port">/dev/ttyUSB0</param>
+                <param name="baud_rate">115200</param>
+            </hardware>
+            <joint name="${left}_joint">
+                <command_interface name="velocity"/>
+                <state_interface name="position"/>
+                <state_interface name="velocity"/>
+            </joint>
+            <joint name="${right}_joint">
+                <command_interface name="velocity"/>
+                <state_interface name="position"/>
+                <state_interface name="velocity"/>
+            </joint>
+        </ros2_control>
+    </xacro:macro>
 </robot>

File: ros2_dual_stepper_controller/description/urdf/dual_stepper.urdf.xacro (robot description, xacro)
@@ -14,8 +14,8 @@
     <!-- Robot structure -->
     <xacro:base_link/>
-    <xacro:wheel wheel_name="left_wheel" parent="base_link"
+    <xacro:wheel name="left_wheel" parent="base_link"
             xyz="-0.1156 0.0 0.046" rpy="0 0 0" axis="1 0 0"/>
-    <xacro:wheel wheel_name="right_wheel" parent="base_link"
+    <xacro:wheel name="right_wheel" parent="base_link"
             xyz="0.1156 0.0 0.046" rpy="0 ${pi} 0" axis="1 0 0"/>
-    <xacro:ros2_dual_stepper_controller name="DualStepperSystem" />
+    <xacro:ros2_dual_stepper_controller name="DualStepperSystem" left="left_wheel" right="right_wheel"/>
 </robot>

File: ros2_dual_stepper_controller/description/urdf/robot_parts/base_link.xacro (robot description, xacro)
@@ -1,21 +1,21 @@
 <?xml version="1.0"?>
 <robot xmlns:xacro="http://ros.org/wiki/xacro">
-<xacro:macro name="base_link" xmlns:xacro="http://ros.org/wiki/xacro">
-    <link name="base_link">
-        <visual>
-            <origin rpy="0.0 0.0 0.0" xyz="0.0 0.0 0.0"/>
-            <geometry>
-                <mesh filename="package://ros2_dual_stepper_controller/description/meshes/urdf_base_link.stl"
-                      scale="1 1 1"/>
-            </geometry>
-            <material name="dark_grey"/>
-        </visual>
-        <!-- Inertial is formally required by ros2_control but not functionally necessary for this simple example-->
-        <inertial>
-            <mass value="0.1"/>
-            <origin xyz="0 0 0" rpy="0 0 0"/>
-            <inertia ixx="1e-6" ixy="0" ixz="0" iyy="1e-6" iyz="0" izz="1e-6"/>
-        </inertial>
-    </link>
-</xacro:macro>
+    <xacro:macro name="base_link">
+        <link name="base_link">
+            <visual>
+                <origin rpy="0.0 0.0 0.0" xyz="0.0 0.0 0.0"/>
+                <geometry>
+                    <mesh filename="package://ros2_dual_stepper_controller/description/meshes/urdf_base_link.STL"
+                          scale="1 1 1"/>
+                </geometry>
+                <material name="dark_grey"/>
+            </visual>
+            <!-- Inertial is formally required by ros2_control but not functionally necessary for this simple example-->
+            <inertial>
+                <mass value="0.1"/>
+                <origin xyz="0 0 0" rpy="0 0 0"/>
+                <inertia ixx="1e-6" ixy="0" ixz="0" iyy="1e-6" iyz="0" izz="1e-6"/>
+            </inertial>
+        </link>
+    </xacro:macro>
 </robot>

File: ros2_dual_stepper_controller/description/urdf/robot_parts/wheel.xacro (robot description, xacro)
@@ -1,27 +1,27 @@
 <?xml version="1.0"?>
 <robot xmlns:xacro="http://ros.org/wiki/xacro">
-<xacro:macro name="wheel" params="wheel_name parent xyz rpy axis" xmlns:xacro="http://ros.org/wiki/xacro">
-    <link name="${wheel_name}">
-        <visual>
-            <origin rpy="0.0 0.0 0.0" xyz="0.0 0.0 0.0"/>
-            <geometry>
-                <mesh filename="package://ros2_dual_stepper_controller/description/meshes/urdf_wheel.stl"
-                      scale="1 1 1"/>
-            </geometry>
-            <material name="grey"/>
-        </visual>
-        <!-- Inertial is formally required by ros2_control but not functionally necessary for this simple example-->
-        <inertial>
-            <mass value="0.1"/>
-            <origin xyz="0 0 0" rpy="0 0 0"/>
-            <inertia ixx="1e-6" ixy="0" ixz="0" iyy="1e-6" iyz="0" izz="1e-6"/>
-        </inertial>
-    </link>
-    <joint name="${wheel_name}_joint" type="continuous">
-        <parent link="${parent}"/>
-        <child link="${wheel_name}"/>
-        <origin xyz="${xyz}" rpy="${rpy}"/>
-        <axis xyz="${axis}"/>
-    </joint>
-</xacro:macro>
+    <xacro:macro name="wheel" params="name parent xyz rpy axis" >
+        <link name="${name}">
+            <visual>
+                <origin rpy="0.0 0.0 0.0" xyz="0.0 0.0 0.0"/>
+                <geometry>
+                    <mesh filename="package://ros2_dual_stepper_controller/description/meshes/urdf_wheel.STL"
+                          scale="1 1 1"/>
+                </geometry>
+                <material name="grey"/>
+            </visual>
+            <!-- Inertial is formally required by ros2_control but not functionally necessary for this simple example-->
+            <inertial>
+                <mass value="0.1"/>
+                <origin xyz="0 0 0" rpy="0 0 0"/>
+                <inertia ixx="1e-6" ixy="0" ixz="0" iyy="1e-6" iyz="0" izz="1e-6"/>
+            </inertial>
+        </link>
+        <joint name="${name}_joint" type="continuous">
+            <parent link="${parent}"/>
+            <child link="${name}"/>
+            <origin xyz="${xyz}" rpy="${rpy}"/>
+            <axis xyz="${axis}"/>
+        </joint>
+    </xacro:macro>
 </robot>
