Commit message: updated xacro file for new meshes

File: ros2_dual_stepper_controller/description/urdf/dual_stepper.urdf.xacro (robot description, xacro)
@@ -15,7 +15,7 @@
     <xacro:base_link/>
     <xacro:wheel name="left_wheel" parent="base_link"
-            xyz="-0.1156 0.0 0.046" rpy="0 0 0" axis="1 0 0"/>
+            xyz="-0.1156 0.0 0.046" rpy="0 0 0" axis="1 0 0" mesh_filename="urdf_left_wheel.STL"/>
     <xacro:wheel name="right_wheel" parent="base_link"
-            xyz="0.1156 0.0 0.046" rpy="0 ${pi} 0" axis="1 0 0"/>
+            xyz="0.1156 0.0 0.046" rpy="0 ${pi} 0" axis="1 0 0" mesh_filename="urdf_right_wheel.STL"/>
     <xacro:ros2_dual_stepper_controller name="DualStepperSystem" left="left_wheel" right="right_wheel"/>
 </robot>

File: ros2_dual_stepper_controller/description/urdf/robot_parts/wheel.xacro (robot description, xacro)
@@ -1,10 +1,10 @@
 <?xml version="1.0"?>
 <robot xmlns:xacro="http://ros.org/wiki/xacro">
-    <xacro:macro name="wheel" params="name parent xyz rpy axis" >
+    <xacro:macro name="wheel" params="name parent xyz rpy axis mesh_filename" >
         <link name="${name}">
             <visual>
                 <origin rpy="0.0 0.0 0.0" xyz="0.0 0.0 0.0"/>
                 <geometry>
-                    <mesh filename="package://ros2_dual_stepper_controller/description/meshes/urdf_wheel.STL"
+                    <mesh filename="package://ros2_dual_stepper_controller/description/meshes/${mesh_filename}"
                           scale="1 1 1"/>
                 </geometry>

Commit message: updated xacro

File: ros2_dual_stepper_controller/description/urdf/dual_stepper.urdf.xacro (robot description, xacro)
@@ -18,5 +18,5 @@
     <xacro:wheel name="right_wheel" parent="base_link"
             xyz="0.0 -0.1175 0.0" rpy="0 0 0" axis="0 1 0" mesh_filename="urdf_right_wheel.STL"/>
-    <xacro:lidar_sensor name="lidar_link" parent="base_link"
+    <xacro:lidar_sensor name="lidar" parent="base_link"
                         xyz="0.29685 0 0.0845" rpy="0 0 0" mesh_filename="urdf_lidar_link.STL"/>
     <xacro:ros2_dual_stepper_controller name="DualStepperSystem" left="left_wheel" right="right_wheel"/>

File: ros2_dual_stepper_controller/description/urdf/robot_parts/base_link.xacro (robot description, xacro)
@@ -4,5 +4,5 @@
         <link name="base_link">
             <visual>
-                <origin rpy="0.0 0.0 0.0" xyz="0.0 0.0475 0.0"/>
+                <origin rpy="0.0 0.0 0.0" xyz="0.0 0.0 0.0475"/>
                 <geometry>
                     <mesh filename="package://ros2_dual_stepper_controller/description/meshes/urdf_base_link.STL"
