Commit message: updated xacro

File: ros2_dual_stepper_controller/description/urdf/robot_parts/base_link.xacro (robot description, xacro)
@@ -1,4 +1,4 @@
 <?xml version="1.0"?>
-<xacro:macro name="base_link" >
+<xacro:macro name="base_link" xmlns:xacro="http://ros.org/wiki/xacro">
     <link name="base_link">
         <visual>

File: ros2_dual_stepper_controller/description/urdf/robot_parts/wheel.xacro (robot description, xacro)
@@ -1,4 +1,4 @@
 <?xml version="1.0"?>
-<xacro:macro name="wheel" params="name parent xyz rpy axis" >
+<xacro:macro name="wheel" params="name parent xyz rpy axis" xmlns:xacro="http://ros.org/wiki/xacro">
     <link name="${name}">
         <visual>

Commit message: modified mesh parameters

File: ros2_dual_stepper_controller/description/urdf/robot_parts/base_link.xacro (robot description, xacro)
@@ -4,5 +4,5 @@
         <link name="base_link">
             <visual>
-                <origin rpy="0.0 0.0 0.0" xyz="0.0 0.0 0.0"/>
+                <origin rpy="0.0 0.0 0.0" xyz="0.0 0.0475 0.0"/>
                 <geometry>
                     <mesh filename="package://ros2_dual_stepper_controller/description/meshes/urdf_base_link.STL"

File: ros2_dual_stepper_controller/description/urdf/robot_parts/lidar.xacro (robot description, xacro)
@@ -8,5 +8,5 @@
                 <origin xyz="0 0 0" rpy="0 0 0"/>
                 <geometry>
-                    <mesh filename="package://my_robot/meshes/${mesh_filename}" scale="1 1 1"/>
+                    <mesh filename="package://ros2_dual_stepper_controller/description/meshes/${mesh_filename}" scale="1 1 1"/>
                 </geometry>
                 <material name="grey"/>

Commit message: removed z offset in base_link

File: ros2_dual_stepper_controller/description/urdf/robot_parts/base_link.xacro (robot description, xacro)
@@ -4,5 +4,5 @@
         <link name="base_link">
             <visual>
-                <origin rpy="0.0 0.0 0.0" xyz="0.0 0.0 0.0475"/>
+                <origin rpy="0.0 0.0 0.0" xyz="0.0 0.0 0.0"/>
                 <geometry>
                     <mesh filename="package://ros2_dual_stepper_controller/description/meshes/urdf_base_link.STL"
